Commit message: update

File: others/test.urdf (robot description, URDF)
Before this commit: robot test_robot, 4 links, 3 joints
Links:
- added link world
- link link3: geometry visual mesh filename=package://ur_description/meshes/ur5/collision/wrist1.stl
- link link4: geometry visual mesh filename=package://ur_description/meshes/ur5/collision/wrist2.stl
Joints:
- added joint world_joint: type fixed, parent world, child link1, origin xyz=0 0 0 rpy=0 0 0
- joint joint1: axis 0 0 1 -> 0 1 0; origin xyz=0.3 0 0.1 rpy=0 0 0 -> xyz=0.6 0 0.1 rpy=0 0 0
