Commit message: update

File: python/myrobot.urdf (robot description, URDF)
Before this commit: robot ur5, 21 links, 20 joints
Links:
- link base_link: geometry collision box size=0.147213 0.183552 0.024058; visual mesh filename=package://ur_description/meshes/ur5/visual/base.dae
- link bh_base_link: geometry collision box size=0.08892 0.06004 0.089018; visual mesh filename=package://barrett_hand_description/meshes/palm_282.dae
- link bh_finger_11_link: geometry collision box size=0.024609 0.048139 0.08193; visual mesh filename=package://barrett_hand_description/meshes/knuckle.dae
- link bh_finger_12_link: geometry collision box size=0.021008 0.025315 0.091919; visual mesh filename=package://barrett_hand_description/meshes/finger.dae
- link bh_finger_13_link: geometry collision box size=0.023012 0.019021 0.06776; visual mesh filename=package://barrett_hand_description/meshes/finger_tip.dae
- link bh_finger_21_link: geometry collision box size=0.024609 0.048139 0.081928; visual mesh filename=package://barrett_hand_description/meshes/knuckle.dae
- link bh_finger_22_link: geometry collision box size=0.021007 0.025315 0.091919; visual mesh filename=package://barrett_hand_description/meshes/finger.dae
- link bh_finger_23_link: geometry collision box size=0.023013 0.019021 0.067759; visual mesh filename=package://barrett_hand_description/meshes/finger_tip.dae
- link bh_finger_31_link: geometry collision box size=0.024006 0.026001 0.042975; visual mesh filename=package://barrett_hand_description/meshes/knuckle_fixed.dae
- link bh_finger_32_link: geometry collision box size=0.021007 0.02532 0.091919; visual mesh filename=package://barrett_hand_description/meshes/finger.dae
- link bh_finger_33_link: geometry collision box size=0.023015 0.019019 0.06774; visual mesh filename=package://barrett_hand_description/meshes/finger_tip.dae
- link forearm_link: geometry collision box size=0.488926 0.111667 0.116547; visual mesh filename=package://ur_description/meshes/ur5/visual/forearm.dae
- link shoulder_link: geometry collision box size=0.118743 0.130248 0.13371; visual mesh filename=package://ur_description/meshes/ur5/visual/shoulder.dae
- link upper_arm_link: geometry collision box size=0.543115 0.133547 0.119571; visual mesh filename=package://ur_description/meshes/ur5/visual/upperarm.dae
- link wrist_1_link: geometry collision box size=0.077432 0.085013 0.104678; visual mesh filename=package://ur_description/meshes/ur5/visual/wrist1.dae
- link wrist_2_link: geometry collision box size=0.077329 0.104691 0.084234; visual mesh filename=package://ur_description/meshes/ur5/visual/wrist2.dae
- link wrist_3_link: geometry collision box size=0.075031 0.034501 0.080516; visual mesh filename=package://ur_description/meshes/ur5/visual/wrist3.dae
